Commit message: urdf changes

File: ros2bot_urdf/urdf/ros2bot.urdf (robot description, URDF)
Before this commit: robot ros2bot, 5 links, 4 joints
Links:
- added link base_footprint
- added link camera_link, mass 0; collision mesh filename=package://yahboomcar_description/meshes/sensor/camera_link.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; visual mesh filename=package://yahboomcar_description/meshes/sensor/camera_link.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
- added link imu_link
- added link laser_link, mass 0.0483909504209895; collision mesh filename=package://yahboomcar_description/meshes/sensor/laser_link.S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; visual mesh filename=package://yahboomcar_description/meshes/sensor/laser_link.S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
- link base_link: mass None -> 0.486218814966626
- link left_front_link: mass None -> 0.051543
- link left_wheel_link: mass None -> 0.0515309299357028
- link right_front_link: mass None -> 0.051532
- link right_wheel_link: mass None -> 0.051540174053366
Joints:
- added joint base_imu: type fixed, parent base_link, child imu_link, origin xyz=-0.06 0.01 0.01 rpy=0 3.1415 1.5707
- added joint base_joint: type fixed, parent base_footprint, child base_link, origin xyz=0.0 0.0 0.0815 rpy=0 0 0
- added joint camera_joint: type fixed, parent base_link, child camera_link, origin xyz=0.057105 1.7948E-05 0.03755 rpy=0 0 0
- added joint laser_joint: type fixed, parent base_link, child laser_link, origin xyz=0.0435 5.25826986680105E-05 0.11 rpy=0 0 0
- joint left_front_joint: limit (none) -> effort=100 velocity=1
- joint left_wheel_joint: limit (none) -> effort=100 velocity=1
- joint right_front_joint: limit (none) -> effort=100 velocity=1
- joint right_wheel_joint: limit (none) -> effort=100 velocity=1

Commit message: urdf changes

File: ros2bot_urdf/urdf/ros2bot.urdf (robot description, URDF)
Before this commit: robot ros2bot, 9 links, 8 joints
Links:
- link camera_link: geometry collision mesh filename=package://ros2bot_urdf/meshes/sensor/camera_link.STL; visual mesh filename=package://ros2bot_urdf/meshes/sensor/camera_link.STL
- link laser_link: geometry collision mesh filename=package://ros2bot_urdf/meshes/sensor/laser_link.STL; visual mesh filename=package://ros2bot_urdf/meshes/sensor/laser_link.STL

Commit message: urdf changes

File: ros2bot_urdf/urdf/ros2bot.urdf (robot description, URDF)
Before this commit: robot ros2bot, 9 links, 8 joints
Links:
- link left_front_link: geometry visual mesh filename=package://ros2bot_urdf/meshes/mecanum/front_left_wheel.STL
- link left_wheel_link: geometry visual mesh filename=package://ros2bot_urdf/meshes/mecanum/back_left_wheel.STL
- link right_front_link: geometry visual mesh filename=package://ros2bot_urdf/meshes/mecanum/front_right_wheel.STL
- link right_wheel_link: geometry visual mesh filename=package://ros2bot_urdf/meshes/mecanum/back_right_wheel.STL
